File: main.sch (EAGLE design)
At the start: 53 parts, among them J1 SJ-3502-SMT-TR, Q1 2N2222A, Q2 2SCR574D3TL1, U1 L78L06ABZ, U3 LM386M-1, Y1 7.040MHz

Commit message: first attempt at board layout
Parts:
- C22: value (none) -> 33u/16V; CAP 33u/16V -> (none)
- Q1: value 2N2222A -> 2SCR574D3TL1; device transistor-npn:2N2222A -> zort2:2SCR574D3TL1
- R2: value (none) -> 1k; device adafruit:R-US_M0805 -> pot:TRIM_EU-3223G
- R3: value 1k -> 6.8k; device pot:TRIM_EU-3223G -> adafruit:R-US_M0805
- U1: value L78L06ABZ -> MCP1703T-5002E; device L78L06ABZ:L78L06ABZ -> linear:MCP170312MB
- X1: value (none) -> Antenna
- renumbered U$1 to U2
Connections:
- net 6V_DC: now also R2.E, U1.VO; no longer R3.E, U1.VOUT
- net GND: now also R2.A, R3.1, X1.GND1, X1.GND2, X1.GND3; no longer R2.1, R3.A
- net N$18: now also R2.S; no longer R3.S
- net N$19: now also Q1.1; no longer Q1.B
- net N$20: now also Q1.3; no longer Q1.E
- net N$21: now also Q1.2; no longer Q1.C
- net N$8: now also R3.2; no longer R2.2
- net VIN: now also U1.VI1; no longer U1.VIN
