File: main.brd (EAGLE design)
At the start: 100 x 80 mm, 53 parts, among them J1 SJ-3502-SMT-TR, Q1 2N2222A, Q2 2SCR574D3TL1, U1 L78L06ABZ, U3 LM386M-1, Y1 7.040MHz

Commit message: first attempt at board layout
Parts:
- removed U$1: SA602AD8-SOIC, zort2:SOIC127P599X175-8N
- added U2: SA602AD8-SOIC, zort2:SOIC127P599X175-8N
- C22: value (none) -> 33u/16V
- Q1: value 2N2222A -> 2SCR574D3TL1; device transistor-npn:TO18 -> zort2:TRANS_2SCR573D_ROM
- R2: value (none) -> 1k; device adafruit:M0805 -> pot:3223G
- R3: value 1k -> 6.8k; device pot:3223G -> adafruit:M0805
- U1: value L78L06ABZ -> MCP1703T-5002E; device L78L06ABZ:TO127P254X749-3 -> linear:SOT89
- X1: value (none) -> Antenna
- moved C10 86.9 mm to (12.7, 5.08), flipped to the bottom
- moved L6 80.4 mm to (6.99, 18.8), turned to 270 degrees
- moved C15 80.2 mm to (9.78, 18.8), turned to 90 degrees
- moved L2 78.4 mm to (17.8, 8.89), flipped to the bottom, turned to 180 degrees
- moved L5 77.4 mm to (14.0, 29.2), flipped to the bottom
- moved Q2 77.1 mm to (17.8, 20.3), flipped to the bottom
- moved L3 74.7 mm to (8.89, 10.2), flipped to the bottom, turned to 90 degrees
- moved C3 74.3 mm to (9.02, 33.7)
- moved C5 72.7 mm to (3.17, 11.7)
- moved L4 71.2 mm to (8.89, 22.9), flipped to the bottom
- moved C9 70.5 mm to (8.89, 25.4), flipped to the bottom
- moved R4 69.2 mm to (9.65, 2.16), flipped to the bottom
- moved C23 68.2 mm to (3.17, 8.51)
- moved C11 67.6 mm to (3.81, 16.5), flipped to the bottom
- moved C2 65.4 mm to (2.54, 27.9), flipped to the bottom, turned to 180 degrees
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Connections:
- removed net GND1: X1.GND@4
- removed net GND2: X1.GND@3
- removed net GND3: X1.GND@2
- net 6V_DC: now also R2.3, U1.3, U2.8; no longer R3.3, U$1.8, U1.1
- net GND: now also U1.1, U2.3, X1.GND@2, X1.GND@3, X1.GND@4; no longer U$1.3, U1.2
- net N$1: now also U2.1; no longer U$1.1
- net N$18: now also R2.2; no longer R3.2
- net N$19: now also Q1.1; no longer Q1.2
- net N$2: now also U2.2; no longer U$1.2
- net N$20: now also Q1.3; no longer Q1.1
- net N$21: now also Q1.2; no longer Q1.3
- net N$4: now also U2.6; no longer U$1.6
- net N$8: now also R3.2, U2.7; no longer R2.2, U$1.7
- net OUT_A: now also U2.4; no longer U$1.4
- net OUT_B: now also U2.5; no longer U$1.5
- net VIN: now also U1.2@1; no longer U1.3
Routing:
- net GND: track 0.00 -> 201.2 mm, vias 0 -> 5
- net 6V_DC: track 0.00 -> 89.8 mm, vias 0 -> 2
- net VIN: track 0.00 -> 81.9 mm, vias 0 -> 5
- net N$19: track 0.00 -> 66.4 mm, vias 0 -> 4
- net N$27: track 0.00 -> 40.0 mm
- net N$8: track 0.00 -> 31.3 mm, vias 0 -> 4
- net OUT_A: track 0.00 -> 27.7 mm, vias 0 -> 3
- net OUT_B: track 0.00 -> 24.3 mm
- net N$14: track 0.00 -> 19.7 mm
- net N$20: track 0.00 -> 16.7 mm
- net N$13: track 0.00 -> 16.1 mm, vias 0 -> 2
- net N$9: track 0.00 -> 15.2 mm
- net N$5: track 0.00 -> 15.2 mm
- net KEY_IN: track 0.00 -> 14.7 mm, vias 0 -> 1
- net N$24: track 0.00 -> 14.6 mm
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Other:
- board size 100 x 80 mm -> 22 x 40 mm

Commit message: splitting boards, doing layouts
Split into two boards with jumpers between. Added jumper for crystal to be able to change reference frequency. Closer to real layouts, still need to solidify some parts.
Connections:
- net N$7 renamed ANT_IN
- net N$8 renamed ANT_OUT
Changed lines of the file:
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@@
 <wire x1="11.5824" y1="23.1648" x2="11.56" y2="23.2" width="0.1524" layer="1"/>
 </signal>
-<signal name="N$7">
-<contactref element="L8" pad="1"/>
-<contactref element="D1" pad="A"/>
-<contactref element="D2" pad="C"/>
+<signal name="ANT_IN">
 <contactref element="C9" pad="2"/>
-<wire x1="16.1544" y1="27.8892" x2="14.0208" y2="27.8892" width="0.1524" layer="1"/>
-<wire x1="16.4592" y1="28.194" x2="16.1544" y2="27.8892" width="0.1524" layer="1"/>
-<wire x1="14.0208" y1="27.8892" x2="13.97" y2="27.845" width="0.1524" layer="1"/>
-<wire x1="16.4592" y1="28.194" x2="16.51" y2="28.3075" width="0.1524" layer="1"/>
-<wire x1="16.6116" y1="28.3464" x2="19.05" y2="28.3464" width="0.1524" layer="1"/>
-<wire x1="19.05" y1="28.3464" x2="19.05" y2="28.3075" width="0.1524" layer="1"/>
-<wire x1="16.6116" y1="28.3464" x2="16.51" y2="28.3075" width="0.1524" layer="1"/>
 <wire x1="8.8392" y1="26.2128" x2="8.0772" y2="25.4508" width="0.1524" layer="16"/>
 <wire x1="8.8392" y1="26.3652" x2="8.8392" y2="26.2128" width="0.1524" layer="16"/>
@@
 <wire x1="13.8684" y1="27.7368" x2="13.4112" y2="27.2796" width="0.1524" layer="1"/>
 <wire x1="8.0772" y1="25.4508" x2="8.04" y2="25.4" width="0.1524" layer="16"/>
-<wire x1="13.8684" y1="27.7368" x2="13.97" y2="27.845" width="0.1524" layer="1"/>
 <via x="11.43" y="27.2796" extent="1-16" drill="0.35"/>
+<contactref element="L8" pad="1"/>
+<contactref element="D1" pad="A"/>
+<contactref element="D2" pad="C"/>
+<wire x1="16.1544" y1="27.8892" x2="14.0208" y2="27.8892" width="0.1524" layer="1"/>
+<wire x1="16.4592" y1="28.194" x2="16.1544" y2="27.8892" width="0.1524" layer="1"/>
+<wire x1="14.0208" y1="27.8892" x2="13.97" y2="27.845" width="0.1524" layer="1"/>
+<wire x1="16.4592" y1="28.194" x2="16.51" y2="28.3075" width="0.1524" layer="1"/>
+<wire x1="16.6116" y1="28.3464" x2="19.05" y2="28.3464" width="0.1524" layer="1"/>
+<wire x1="19.05" y1="28.3464" x2="19.05" y2="28.3075" width="0.1524" layer="1"/>
+<wire x1="16.6116" y1="28.3464" x2="16.51" y2="28.3075" width="0.1524" layer="1"/>
+<wire x1="13.8684" y1="27.7368" x2="13.97" y2="27.845" width="0" layer="19" extent="1-1"/>
 </signal>
 <signal name="OUT_A">
@@
 <wire x1="2.4384" y1="22.098" x2="2.325" y2="21.971" width="0.1524" layer="1"/>
 </signal>
-<signal name="N$8">
+<signal name="ANT_OUT">
 <contactref element="U2" pad="7"/>
 <contactref element="C14" pad="2"/>
 <contactref element="C13" pad="1"/>
 <contactref element="R3" pad="2"/>
-<contactref element="C12" pad="1"/>
 <wire x1="19.9644" y1="16.9164" x2="19.9644" y2="14.3256" width="0.1524" layer="1"/>
 <wire x1="19.9644" y1="14.3256" x2="19.9" y2="14.224" width="0.1524" layer="1"/>
@@
 <wire x1="4.2672" y1="21.7932" x2="5.7912" y2="21.7932" width="0.1524" layer="1"/>
 <wire x1="4.1148" y1="21.9456" x2="4.2672" y2="21.7932" width="0.1524" layer="1"/>
-<wire x1="4.7244" y1="22.86" x2="4.66" y2="22.86" width="0.1524" layer="16"/>
 <wire x1="4.1148" y1="21.9456" x2="4.025" y2="21.971" width="0.1524" layer="1"/>
 <wire x1="18.5928" y1="17.0688" x2="19.9644" y2="17.0688" width="0.1524" layer="1"/>
@@
 <via x="14.3256" y="24.0792" extent="1-16" drill="0.35"/>
 <via x="9.144" y="21.1836" extent="1-16" drill="0.35"/>
+<contactref element="C12" pad="1"/>
+<wire x1="4.7244" y1="22.86" x2="4.66" y2="22.86" width="0" layer="19" extent="16-16"/>
 </signal>
 <signal name="N$15">

Commit message: updating layouts and parts
Connections:
- net ANT_IN renamed N$7
- net ANT_OUT renamed N$8
Routing:
- net N$27: track 40.0 -> 0.00 mm
Changed lines of the file:
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@@
 <wire x1="22.00000625" y1="39.99991875" x2="0" y2="39.99991875" width="0" layer="20"/>
 <wire x1="0" y1="39.99991875" x2="0" y2="0" width="0" layer="20"/>
+<wire x1="22.00000625" y1="0" x2="22.00000625" y2="39.99991875" width="0" layer="20"/>
 </plain>
 <attributes>
@@
 <wire x1="11.5824" y1="23.1648" x2="11.56" y2="23.2" width="0.1524" layer="1"/>
 </signal>
-<signal name="ANT_IN">
+<signal name="N$7">
+<contactref element="L8" pad="1"/>
+<contactref element="D1" pad="A"/>
+<contactref element="D2" pad="C"/>
 <contactref element="C9" pad="2"/>
+<wire x1="16.1544" y1="27.8892" x2="14.0208" y2="27.8892" width="0.1524" layer="1"/>
+<wire x1="16.4592" y1="28.194" x2="16.1544" y2="27.8892" width="0.1524" layer="1"/>
+<wire x1="14.0208" y1="27.8892" x2="13.97" y2="27.845" width="0.1524" layer="1"/>
+<wire x1="16.4592" y1="28.194" x2="16.51" y2="28.3075" width="0.1524" layer="1"/>
+<wire x1="16.6116" y1="28.3464" x2="19.05" y2="28.3464" width="0.1524" layer="1"/>
+<wire x1="19.05" y1="28.3464" x2="19.05" y2="28.3075" width="0.1524" layer="1"/>
+<wire x1="16.6116" y1="28.3464" x2="16.51" y2="28.3075" width="0.1524" layer="1"/>
 <wire x1="8.8392" y1="26.2128" x2="8.0772" y2="25.4508" width="0.1524" layer="16"/>
 <wire x1="8.8392" y1="26.3652" x2="8.8392" y2="26.2128" width="0.1524" layer="16"/>
@@
 <wire x1="13.8684" y1="27.7368" x2="13.4112" y2="27.2796" width="0.1524" layer="1"/>
 <wire x1="8.0772" y1="25.4508" x2="8.04" y2="25.4" width="0.1524" layer="16"/>
+<wire x1="13.8684" y1="27.7368" x2="13.97" y2="27.845" width="0.1524" layer="1"/>
 <via x="11.43" y="27.2796" extent="1-16" drill="0.35"/>
-<contactref element="L8" pad="1"/>
-<contactref element="D1" pad="A"/>
-<contactref element="D2" pad="C"/>
-<wire x1="16.1544" y1="27.8892" x2="14.0208" y2="27.8892" width="0.1524" layer="1"/>
-<wire x1="16.4592" y1="28.194" x2="16.1544" y2="27.8892" width="0.1524" layer="1"/>
-<wire x1="14.0208" y1="27.8892" x2="13.97" y2="27.845" width="0.1524" layer="1"/>
-<wire x1="16.4592" y1="28.194" x2="16.51" y2="28.3075" width="0.1524" layer="1"/>
-<wire x1="16.6116" y1="28.3464" x2="19.05" y2="28.3464" width="0.1524" layer="1"/>
-<wire x1="19.05" y1="28.3464" x2="19.05" y2="28.3075" width="0.1524" layer="1"/>
-<wire x1="16.6116" y1="28.3464" x2="16.51" y2="28.3075" width="0.1524" layer="1"/>
-<wire x1="13.8684" y1="27.7368" x2="13.97" y2="27.845" width="0" layer="19" extent="1-1"/>
 </signal>
 <signal name="OUT_A">
@@
 <wire x1="2.4384" y1="22.098" x2="2.325" y2="21.971" width="0.1524" layer="1"/>
 </signal>
-<signal name="ANT_OUT">
+<signal name="N$8">
 <contactref element="U2" pad="7"/>
 <contactref element="C14" pad="2"/>
 <contactref element="C13" pad="1"/>
 <contactref element="R3" pad="2"/>
+<contactref element="C12" pad="1"/>
 <wire x1="19.9644" y1="16.9164" x2="19.9644" y2="14.3256" width="0.1524" layer="1"/>
 <wire x1="19.9644" y1="14.3256" x2="19.9" y2="14.224" width="0.1524" layer="1"/>
@@
 <wire x1="4.2672" y1="21.7932" x2="5.7912" y2="21.7932" width="0.1524" layer="1"/>
 <wire x1="4.1148" y1="21.9456" x2="4.2672" y2="21.7932" width="0.1524" layer="1"/>
+<wire x1="4.7244" y1="22.86" x2="4.66" y2="22.86" width="0.1524" layer="16"/>
 <wire x1="4.1148" y1="21.9456" x2="4.025" y2="21.971" width="0.1524" layer="1"/>
 <wire x1="18.5928" y1="17.0688" x2="19.9644" y2="17.0688" width="0.1524" layer="1"/>
@@
 <via x="14.3256" y="24.0792" extent="1-16" drill="0.35"/>
 <via x="9.144" y="21.1836" extent="1-16" drill="0.35"/>
-<contactref element="C12" pad="1"/>
-<wire x1="4.7244" y1="22.86" x2="4.66" y2="22.86" width="0" layer="19" extent="16-16"/>
 </signal>
 <signal name="N$15">
@@
 <via x="16.6116" y="32.766" extent="1-16" drill="0.35"/>
 </signal>
-<signal name="N$27">
-<wire x1="22.00000625" y1="0" x2="22.00000625" y2="39.99991875" width="0" layer="16"/>
-</signal>
 </signals>
